File: PS10_DAN_W_89/PS10_DAN_W_89.kicad_sch (KiCad schematic)
At the start: 13 parts, among them J1 Conn_01x15_Pin, J2 IDC26, Q1 BUZ11F1 x 2pcs., Q2 BUZ11F1 x 2pcs., Q3 BUZ11F1 x 2pcs., Q4 BUZ11F1 x 2pcs.

Commit message: Documentation cont.
Parts:
- removed RN1: R_Network09_US, Resistor_THT:R_Array_SIP10, symbol Device:R_Network09_US
- added U1: AD7545, symbol kpole:AD7545
Connections:
- net at J2.10 (Pin_10): now also U1.10 (DB5)
- net at J2.11 (Pin_11): now also U1.12 (DB3)
- net at J2.12 (Pin_12): now also U1.9 (DB6)
- net at J2.13 (Pin_13): now also U1.13 (DB2)
- net at J2.14 (Pin_14): now also U1.8 (DB7)
- net at J2.15 (Pin_15): now also U1.14 (DB1)
- net at J2.16 (Pin_16): now also U1.7 (DB8)
- net at J2.17 (Pin_17): now also U1.15 (DB0)
- net at J2.18 (Pin_18): now also U1.6 (DB9)
- net at J2.19 (Pin_19): now also U1.4 (DB11)
- net at J2.20 (Pin_20): now also U1.5 (DB10)
- net at J2.9 (Pin_9): now also U1.11 (DB4)
Other:
- moved on the sheet: C1, C2, C3, C4, C5, J1, J2, L1, Q1, Q2, Q3, Q4

Commit message: Documentation cont.
Parts:
- added SW1: SW_DIP_x08, symbol Switch:SW_DIP_x08
- added U2, U3: MC14585, symbol kpole:MC14585
- added U7: 74HC14, symbol 74xx:74HC14
Connections:
- net GND: now also J2.23 (Pin_23), J2.24 (Pin_24), SW1.10, SW1.11, SW1.12, SW1.13, SW1.14, SW1.15, SW1.16, SW1.9
- net at U1.16 (~{CS}): now also U7.2
- net at U1.17 (~{WR}): now also J2.21 (Pin_21), J2.22 (Pin_22)
- net at J2.1 (Pin_1): now also U3.7 (A1)
- net at J2.2 (Pin_2): now also U3.2 (A2)
- net at J2.3 (Pin_3): now also U3.15 (A3)
- net at J2.4 (Pin_4): now also U3.10 (A0)
- net at J2.5 (Pin_5): now also U2.7 (A1)
- net at J2.6 (Pin_6): now also U2.2 (A2)
- net at J2.7 (Pin_7): now also U2.15 (A3)
- net at J2.8 (Pin_8): now also U2.10 (A0)
- new net: SW1.4, U2.1 (B2)
- new net: SW1.2, U2.11 (B0)
- new net: SW1.3, U2.14 (B3)
- new net: U2.3 ((A=B)out), U7.1
- new net: U2.6 ((A=B)in), U3.3 ((A=B)out)
- new net: SW1.1, U2.9 (B1)
- new net: SW1.5, U3.9 (B1)
- new net: SW1.6, U3.11 (B0)
- new net: SW1.7, U3.14 (B3)
- new net: SW1.8, U3.1 (B2)
Other:
- moved on the sheet: U1

Commit message: Documentation cont. (schematics)
Parts:
- added C6: 33p, symbol Device:C_Small
- added C7: 47n, symbol Device:C_Small
- added C8: ?, symbol Device:C_Small
- added J100: Sensor_LEM, symbol Connector_Generic:Conn_01x03
- added J101: Conn_01x07, symbol Connector_Generic:Conn_01x07
- added R1: ?, symbol Device:R
- added R10: 4k99, symbol Device:R
- added R11: 1k24, symbol Device:R
- added R21: 10k, symbol Device:R
- added R3: 7k5, symbol Device:R
- added R4: 51k6, symbol Device:R
- added R5: 22k, symbol Device:R
- added R9: 2k55, symbol Device:R
- added RV1: 2k, symbol Device:R_Potentiometer
- added RV2: 500k ?, symbol Device:R_Potentiometer
- added U10, U4: LF353N, symbol Device:Opamp_Dual
- added U14, U6, U8: OP77, symbol Amplifier_Operational:OP77
- added U5: LM399, Package_TO_SOT_THT:Analog_TO-46-4_ThermalShield, symbol Reference_Voltage:LM399
Connections:
- net GND: now also U1.2 (AGND), U1.3 (DGND), U2.8 (VSS), U3.8 (VSS), R11.2, R4.1, U5.2, U8.3 (+); no longer C2.2, C3.2, C4.2, C5.2, J1.12 (Pin_12), J1.14 (Pin_14), J1.5 (Pin_5), J1.6 (Pin_6), J1.7 (Pin_7)
- net at SW1.4, U2.1 (B2): now also J2.6 (Pin_6), U2.2 (A2)
- net at J2.8 (Pin_8), U2.10 (A0): now also SW1.2, U2.11 (B0)
- net Vcc: now reaches U2.16 (VDD)
- net Vcc: now also C5.1, J1.1 (Pin_1), U1.18 (VDD), U3.16 (VDD), J100.3 (Pin_3), R3.1, U14.7 (V+), U4.8 (V+), U5.3, U6.7 (V+), U8.7 (V+)
- net at U1.1 (OUT1): now also C6.2, U8.2 (-)
- net at J2.10 (Pin_10), U1.10 (DB5): now also J2.11 (Pin_11), J2.12 (Pin_12), J2.13 (Pin_13), J2.14 (Pin_14), J2.15 (Pin_15), J2.16 (Pin_16), J2.17 (Pin_17), J2.18 (Pin_18), J2.19 (Pin_19), J2.20 (Pin_20), J2.9 (Pin_9), U1.11 (DB4), U1.12 (DB3), U1.13 (DB2), U1.14 (DB1), U1.15 (DB0), U1.16 (~{CS}), U1.4 (DB11), U1.5 (DB10), U1.6 (DB9), U1.7 (DB8), U1.8 (DB7), U1.9 (DB6), U7.2
- net at U1.19 (VREF): now also R10.1, U14.2 (-), U14.6
- net at U1.20 (RFB): now also C6.1, R9.2, RV2.1, RV2.2, U8.6
- net Vee: now reaches J1.2 (Pin_2)
- net Vee: now also J100.2 (Pin_2), U14.4 (V-), U4.4 (V-), U6.4 (V-), U8.4 (V-)
- new net: R3.2, R5.2, U5.1
- new net: R5.1, RV1.1
- new net: RV1.2, U14.3 (+)
- new net: R4.2, RV1.3
- new net: C7.2, R21.1
- new net: R1.2, R21.2, U6.6
- new net: C8.2, R1.1
- new net: C7.1, C8.1, R10.2, R9.1, RV2.3, U6.2 (-)
- new net: R11.1, U6.3 (+)
- new net Gnd: C2.2, C3.2, C4.2, C5.2, J1.12 (Pin_12), J1.14 (Pin_14), J1.5 (Pin_5), J1.6 (Pin_6), J1.7 (Pin_7)
Other:
- moved on the sheet: C2, C3, C4, C5, J2, SW1, U1, U2, U3, U7A

Commit message: Documentation cont. (schematics)
Parts:
- added Q5: VN10KM, symbol Device:Q_NMOS_SGD
- added R16, R22: 10k, symbol Device:R
- added R17, R18: 309R, symbol Device:R
- added R19: 301R, symbol Device:R
- added R20: 4k99, symbol Device:R
- added R21, R23: 2k49, symbol Device:R
- added R30: 1R, 5%, symbol Device:R
- added U11: LF355N, symbol Amplifier_Operational:AD817
- added U12, U13: LM311, symbol Comparator:LM311
- added U14: CNX38, Package_DIP:DIP-6_W7.62mm, symbol Isolator:4N25
- added U4: MC14013B, symbol kpole:MC14013B
- added U6: MC14011B, symbol 4xxx:4011
- added unit 7 of U7
- J101: value Conn_01x07 -> ?
- Q1, Q2, Q3, Q4: value BUZ11F1 x 2pcs. -> 2 x BUZ11F1
- U7: value 74HC14 -> MC14584B
- renumbered C8 to C7b, R1 to R21b, U4 to U10, U6 to U9
Connections:
- net Gnd is gone; now on net GND: C2.2, C3.2, C4.2, C5.2, J1.12 (Pin_12), J1.14 (Pin_14), J1.5 (Pin_5), J1.6 (Pin_6), J1.7 (Pin_7)
- net GND: now also R17.1, R18.1, R19.1, U12.1 (GND), U13.1 (GND), U7.7 (GND)
- net Vcc: now also J100.1 (Pin_1), J101.1 (Pin_1), R21.2, U12.8 (V+), U13.8 (V+), U7.14 (VCC); no longer J100.3 (Pin_3)
- net Vee: now also J101.4 (Pin_4), R22.1, U12.4 (V-), U13.4 (V-)
- net Out2: now reaches C1.2, J1.8 (Pin_8), J1.9 (Pin_9)
- net at U2.3 ((A=B)out): now also U7.9, Q5.2 (G); no longer U7.1
- net Vpwr: now reaches C2.1, C3.1, C4.1, J1.13 (Pin_13), J1.15 (Pin_15)
- net at R21.2, R21b.2, U9.6: now also R30.2
- net at C7.1, C7b.1, R10.2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: now also R20.2
- net at J101.2 (Pin_2): now also J1.4 (Pin_4), J101.6 (Pin_6)
- net at J101.5 (Pin_5): now also R16.1
- net Out1: now reaches L1.1
- net at J2.25 (Pin_25): now also Q5.3 (D)
- net at J1.3 (Pin_3): now also U6.1, U6.2
- new net: Q5.1 (S), U12.7, U13.7
- new net: J100.3 (Pin_3), R16.2, R17.2, R18.2, R19.2, R20.1
- new net: R30.1, U12.2 (+), U13.2 (+)
- new net: R21.1, R23.2, U13.3 (-)
- new net: U13.5 (BAL), U13.6 (STRB)
- new net: R22.2, R23.1, U12.3 (-)
- new net: U12.5 (BAL), U12.6 (STRB)
- new net: J2.10 (Pin_10), U1.10 (DB5)
- new net: J2.9 (Pin_9), U1.11 (DB4)
- new net: J2.11 (Pin_11), U1.12 (DB3)
- new net: J2.13 (Pin_13), U1.13 (DB2)
- new net: J2.15 (Pin_15), U1.14 (DB1)
- new net: J2.17 (Pin_17), U1.15 (DB0)
- new net: U1.16 (~{CS}), U7.8
- new net: J2.19 (Pin_19), U1.4 (DB11)
- new net: J2.20 (Pin_20), U1.5 (DB10)
- new net: J2.18 (Pin_18), U1.6 (DB9)
- new net: J2.16 (Pin_16), U1.7 (DB8)
- new net: J2.14 (Pin_14), U1.8 (DB7)
- new net: J2.12 (Pin_12), U1.9 (DB6)
Other:
- moved on the sheet: C7, J2, Q1, Q2, Q3, Q4, R10, R11, R21, U10A, U10B, U10C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

Commit message: Schematics cont.
Parts:
- added C8: 18p ?, symbol Device:C_Small
- added D2, D3, D4, D5: D_Small, symbol Device:D_Small
- added R12: 3k6, symbol Device:R
- added R13: 100k, symbol Device:R
- added R14: 220k, symbol Device:R
- added R15, R2: 1k, symbol Device:R
- added R6, R7: 1R, symbol Device:R
- added R8: 100k, 1%, 50ppm, symbol Device:R
- added U15: MC14584B, symbol 74xx:74HC14
- added unit 3 of U5
- added unit 2 of U5
- added unit 1 of U7
- added unit 6 of U7
Connections:
- net GND: now also U4.7 (VSS), U6.7 (VSS), C8.2, D2.1 (K), D4.2 (A), R15.1, U5.7 (VSS)
- net Vcc: now also U11.7 (V+), U4.14 (VDD), U6.14 (VDD), U5.14 (VDD)
- net Vee: now also U11.4 (V-)
- net at R21.2, R21b.2, R30.2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: now also R12.1
- net at U4.10 (R): now also U4.8 (S), U15.6
- net at U4.11 (C): now also U4.3 (C), U5.11 (C), U5.3 (C), U7.12
- net at U4.12 (~{Q}): now also U4.9 (D)
- net at U4.1 (Q): now also U4.5 (D)
- net at U4.4 (R): now also U4.6 (S), R8.2, U15.5
- net at U14.1: now also D4.1 (K), D5.1 (K)
- net at U14.2: now also D2.2 (A), D3.2 (A)
- net at U11.2 (-): now also D3.1 (K), D5.2 (A), R12.2
- net at U11.3 (+): now also R14.1, R15.2
- net at U11.6: now also R13.2, R14.2, R8.1
- new net: R6.2, U5.10 (R), U5.8 (S)
- new net: R7.2, U5.4 (R), U5.6 (S)
- new net: C8.1, R2.1, U7.1
- new net: R2.2, U7.13, U7.2
- new net: U5.12 (~{Q}), U5.9 (D)
- new net: U5.2 (~{Q}), U5.5 (D)
Other:
- moved on the sheet: Q1, Q2, Q3, Q4, U10A, U10B, U11, U14, U4A, U4B, U4C, U6B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

Commit message: Documentation cont. (schematics; datasheet)
Parts:
- removed J101: ?, symbol Connector_Generic:Conn_01x07
- added U16: OP77, symbol Amplifier_Operational:OP77
Connections:
- net Vcc: now also U16.7 (V+)
- net Vee: now also U16.4 (V-)
- net at J100.3 (Pin_3), R17.2, R18.2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: now also R16.1; no longer R16.2
- net LIMIT2: now reaches R21.1, R23.2, U13.3 (-)
- net at R21.2, R21b.2, R30.2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: now also R12.2; no longer R12.1
- net at D3.1 (K), D5.2 (A), U11.2 (-): now also R12.1; no longer R12.2
- net LIMIT1: now reaches R22.2, R23.1, U12.3 (-)
- net at J1.4 (Pin_4): now also U16.2 (-), U16.6
- new net: R16.2, U16.3 (+)
Other:
- moved on the sheet: C1, C2, C3, C4, C5, C6, C7, C7b, C8, D2, D3, D4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

Commit message: Documentation cont. (schematics)
Parts:
- added C8: 22n, symbol Device:C_Small
- added C9: ??, symbol Device:C_Small
- added D1: D_Small, symbol Device:D_Small
- added R24: 1Meg, symbol Device:R
- added R25, R26: 5k76, symbol Device:R
- added R27: 10k, symbol Device:R
- added R28: 18k, symbol Device:R
- added R29: 100R, symbol Device:R
- added R31: 27k, symbol Device:R
- added R32: 120k?, symbol Device:R
Connections:
- net GND: now also U10.3 (+), R24.2, R32.2
- net Vcc: now also R29.2
- net Vee: now also R31.1
- net at U10.5 (+): now also U14.4, R31.2, R32.1
- net at U10.6 (-): now also R28.2
- net at U10.7: now also R27.1
- net at R6.1: now also U6.11
- net at R7.1: now also U6.4
- net BLOCK: now reaches J1.3 (Pin_3), U6.1, U6.2
- net at U6.3: now also R26.1
- net at U6.10: now also U6.12
- net at U6.8: now also R13.1, U6.5, U6.9
- net at U6.13: now also U6.6, R27.2
- net at U14.5: now also R29.1
- net at U10.1: now also C9.2, R28.1
- net at U10.2 (-): now also C8.2, C9.1, R24.1
- new net: C8.1, D1.2 (A), R25.2
- new net: D1.1 (K), R25.1, R26.2
Other:
- moved on the sheet: C8, D2, D3, D4, D5, Q1, Q2, Q3, Q4, R13, R2, R6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

Commit message: Schematics completed; 2 datasheets added;
Parts:
- C9: value ?? -> ?
Connections:
- net Out1 is gone; now on net Out+: L1.1
- net Out2 is gone; now on net Out-: C1.2, J1.8 (Pin_8), J1.9 (Pin_9)
- net Vpwr is gone; now on net Vin: C2.1, C3.1, C4.1, J1.13 (Pin_13), J1.15 (Pin_15)
- net GND: now also Q2.3 (S), Q4.3 (S)
- net IsolatingConverter1/Input+: now reaches U4.12 (~{Q}), U4.9 (D)
- net IsolatingConverter1/Input-: now reaches U4.13 (Q)
- net Out+: now reaches Q4.1 (D)
- net Out+: now also Q3.3 (S)
- net IsolatingConverter3/Output+: now reaches Q4.2 (G)
- net IsolatingConverter/Input+: now reaches U4.1 (Q), U4.5 (D)
- net IsolatingConverter/Input-: now reaches U4.2 (~{Q})
- net Out-: now reaches Q2.1 (D)
- net Out-: now also Q1.3 (S)
- net IsolatingConverter1/Output+: now reaches Q2.2 (G)
- net Vin: now reaches Q3.1 (D)
- net Vin: now also Q1.1 (D)
- net IsolatingConverter2/Output+: now reaches Q3.2 (G)
- net IsolatingConverter/Output+: now reaches Q1.2 (G)
- net IsolatingConverter3/Input+: now reaches U5.12 (~{Q}), U5.9 (D)
- net IsolatingConverter3/Input-: now reaches U5.13 (Q)
- net IsolatingConverter2/Input+: now reaches U5.1 (Q)
- net IsolatingConverter2/Input-: now reaches U5.2 (~{Q}), U5.5 (D)
- net BLOCK renamed SIG1
Other:
- added sheet IsolatingConverter (IsolatingConverter.kicad_sch)
- added sheet IsolatingConverter1 (IsolatingConverter.kicad_sch)
- added sheet IsolatingConverter2 (IsolatingConverter.kicad_sch)
- added sheet IsolatingConverter3 (IsolatingConverter.kicad_sch)
- moved on the sheet: C8, Q1, Q2, Q3, Q4, R2, R8, U15C, U4A, U7A, U7F
